Commit message: rs_desc: use RS080N macro in top-level xacro.

File: rs_description/urdf/rs080n.urdf.xacro (robot description, xacro)
@@ -1,63 +1,7 @@
-<?xml version="1.0"?>
+<?xml version="1.0" ?>
 <robot name="rs080n" xmlns:xacro="http://ros.org/wiki/xacro">
-  <xacro:include filename="$(find rs_description)/urdf/rs.transmission.xacro" />
-  <xacro:include filename="$(find rs_description)/urdf/common.gazebo.xacro" />
-  <!-- mathematics value-->
-  <xacro:property name="pi" value="3.14159265359" />
-  <!-- link rviz colors -->
-  <material name="White">
-    <color rgba="1 1 1 1"/>
-  </material>
-  <material name="Black">
-    <color rgba="0 0 0 1"/>
-  </material>
-  <!-- DH parameters -->
-  <xacro:property name="dh_j1_j2_roty" value="-${pi/2}"/>
-  <xacro:property name="dh_j3_j4_roty" value="${pi/2}"/>
-  <xacro:property name="dh_j4_j5_roty" value="-${pi/2}"/>
-  <xacro:property name="dh_j5_j6_roty" value="${pi/2}"/>
-  <!-- link mass [kg] -->
-  <xacro:property name="j0_mass" value="200"/> <!-- TO-DO -->
-  <xacro:property name="j1_mass" value="216.150"/>
-  <xacro:property name="j2_mass" value="70.847"/>
-  <xacro:property name="j3_mass" value="51.71"/>
-  <xacro:property name="j4_mass" value="31.6751"/>
-  <xacro:property name="j5_mass" value="6.866"/>
-  <xacro:property name="j6_mass" value="0.625"/> <!-- TO-DO -->
-  <!-- link lengths [m] -->
-  <xacro:property name="j0_length" value="0.68"/>
-  <xacro:property name="j1_length" value="0.15"/>
-  <xacro:property name="j2_length" value="0.87"/>
-  <xacro:property name="j3_length" value="0.267"/>
-  <xacro:property name="j4_length" value="0.813"/>
-  <xacro:property name="j5_length" value="0.165"/>
-  <!-- joint limits [rad] -->
-  <xacro:property name="j1_lower_limit" value="${-pi}"/>
-  <xacro:property name="j1_upper_limit" value="${pi}"/>
-  <xacro:property name="j2_lower_limit" value="${-pi*105/180}"/>
-  <xacro:property name="j2_upper_limit" value="${pi*140/180}"/>
-  <xacro:property name="j3_lower_limit" value="${-pi*155/180}"/>
-  <xacro:property name="j3_upper_limit" value="${pi*135/180}"/>
-  <xacro:property name="j4_lower_limit" value="${-pi*360/180}"/>
-  <xacro:property name="j4_upper_limit" value="${pi*360/180}"/>
-  <xacro:property name="j5_lower_limit" value="${-pi*145/180}"/>
-  <xacro:property name="j5_upper_limit" value="${pi*145/180}"/>
-  <xacro:property name="j6_lower_limit" value="${-pi*360/180}"/>
-  <xacro:property name="j6_upper_limit" value="${pi*360/180}"/>
-  <!-- joint velocity limits [rad/s] -->
-  <xacro:property name="j1_velocity_limit" value="${pi*180/180}"/>
-  <xacro:property name="j2_velocity_limit" value="${pi*180/180}"/>
-  <xacro:property name="j3_velocity_limit" value="${pi*160/180}"/>
-  <xacro:property name="j4_velocity_limit" value="${pi*185/180}"/>
-  <xacro:property name="j5_velocity_limit" value="${pi*165/180}"/>
-  <xacro:property name="j6_velocity_limit" value="${pi*280/180}"/>
-  <!-- link inertial(TODO : set correct link inertial )-->
-  <xacro:macro name="default_inertial" params="mass">
-    <inertial>
-      <mass value="${mass}" />
-      <inertia ixx="1.0" ixy="0.0" ixz="0.0" iyy="1.0" iyz="0.0" izz="1.0" />
-    </inertial>
-  </xacro:macro>
-  <!-- rs080n start -->
+  <xacro:include filename="$(find rs_description)/urdf/rs080n_macro.xacro"/>
+  <!-- instantiate rs080n -->
+  <xacro:rs080n />
   <!-- Fix rs080n to world -->
   <link name="world"/>
@@ -67,177 +11,3 @@
     <origin rpy="0 0 0" xyz="0 0 0"/>
   </joint>
-  <!-- Link 0 -->
-  <link name="base_link">
-    <visual>
-      <geometry>
-        <mesh filename="package://rs_description/meshes/RS080N_J0.stl"/>
-      </geometry>
-      <material name="White"/>
-      <origin rpy="0 0 0" xyz="0 0 0"/>
-    </visual>
-    <collision>
-      <geometry>
-        <mesh filename="package://rs_description/meshes/RS080N_J0.stl"/>
-      </geometry>
-      <material name="White"/>
-      <origin rpy="0 0 0" xyz="0 0 0"/>
-    </collision>
-    <xacro:default_inertial mass="${j0_mass}"/>
-  </link>
-  <!-- Link 1 -->
-  <joint name="joint1" type="revolute">
-    <axis xyz="0 0 -1" rpy="0 0 0" />
-    <limit effort="1000.0" lower="${j1_lower_limit}" upper="${j1_upper_limit}" velocity="${j1_velocity_limit}"/>
-    <origin xyz="0 0 ${j0_length}" rpy="0 0 0" />
-    <parent link="base_link"/>
-    <child link="link1"/>
-    <dynamics damping="0.0" friction="0.0"/>
-  </joint>
-  <link name="link1">
-    <visual>
-      <geometry>
-        <mesh filename="package://rs_description/meshes/RS080N_J1.stl"/>
-      </geometry>
-      <material name="White"/>
-      <origin rpy="0 0 0" xyz="0 0 0"/>
-    </visual>
-    <collision>
-      <geometry>
-        <mesh filename="package://rs_description/meshes/RS080N_J1.stl"/>
-      </geometry>
-      <material name="White"/>
-      <origin rpy="0 0 0" xyz="0 0 0"/>
-    </collision>
-    <xacro:default_inertial mass="${j1_mass}"/>
-  </link>
-  <!-- Link 2 -->
-  <joint name="joint2" type="revolute">
-    <axis xyz="0 0 1" rpy="0 0 0" />
-    <limit effort="1000.0" lower="${j2_lower_limit}" upper="${j2_upper_limit}" velocity="${j2_velocity_limit}"/>
-    <origin xyz="0 ${j1_length} 0" rpy="0 ${dh_j1_j2_roty} 0" />
-    <parent link="link1"/>
-    <child link="link2"/>
-    <dynamics damping="0.0" friction="0.0"/>
-  </joint>
-  <link name="link2">
-    <visual>
-      <geometry>
-        <mesh filename="package://rs_description/meshes/RS080N_J2.stl"/>
-      </geometry>
-      <material name="White"/>
-      <origin xyz="0 0 0" rpy="0 ${dh_j1_j2_roty*-1} 0"/>
-    </visual>
-    <collision>
-      <geometry>
-        <mesh filename="package://rs_description/meshes/RS080N_J2.stl"/>
-      </geometry>
-      <material name="White"/>
-      <origin xyz="0 0 0" rpy="0 ${dh_j1_j2_roty*-1} 0"/>
-    </collision>
-    <xacro:default_inertial mass="${j2_mass}"/>
-  </link>
-  <!-- Link 3 -->
-  <joint name="joint3" type="revolute">
-    <axis xyz="0 0 -1" rpy="0 0 0" />
-    <limit effort="1000.0" lower="${j3_lower_limit}" upper="${j3_upper_limit}" velocity="${j3_velocity_limit}"/>
-    <origin xyz="${j2_length} 0 0" rpy="0 0 0" />
-    <parent link="link2"/>
-    <child link="link3"/>
-    <dynamics damping="0.0" friction="0.0"/>
-  </joint>
-  <link name="link3">
-    <visual>
-      <geometry>
-        <mesh filename="package://rs_description/meshes/RS080N_J3.stl"/>
-      </geometry>
-      <material name="White"/>
-      <origin xyz="0 0 0" rpy="0 ${dh_j1_j2_roty*-1} 0"/>
-    </visual>
-    <collision>
-      <geometry>
-        <mesh filename="package://rs_description/meshes/RS080N_J3.stl"/>
-      </geometry>
-      <material name="White"/>
-      <origin xyz="0 0 0" rpy="0 ${dh_j1_j2_roty*-1} 0"/>
-    </collision>
-    <xacro:default_inertial mass="${j3_mass}"/>
-  </link>
-  <!-- Link 4 -->
-  <joint name="joint4" type="revolute">
-    <axis xyz="0 0 1" rpy="0 0 0" />
-    <limit effort="1000.0" lower="${j4_lower_limit}" upper="${j4_upper_limit}" velocity="${j4_velocity_limit}"/>
-    <origin xyz="${j3_length} 0 0" rpy="0 ${dh_j3_j4_roty} 0" />
-    <parent link="link3"/>
-    <child link="link4"/>
-    <dynamics damping="0.0" friction="0.0"/>
-  </joint>
-  <link name="link4">
-    <visual>
-      <geometry>
-        <mesh filename="package://rs_description/meshes/RS080N_J4.stl"/>
-      </geometry>
-      <material name="White"/>
-      <origin xyz="0 0 ${j4_length}" rpy="0 0 0"/>
-    </visual>
-    <collision>
-      <geometry>
-        <mesh filename="package://rs_description/meshes/RS080N_J4.stl"/>
-      </geometry>
-      <material name="White"/>
-      <origin xyz="0 0 ${j4_length}" rpy="0 0 0"/>
-    </collision>
-    <xacro:default_inertial mass="${j4_mass}"/>
-  </link>
-  <!-- Link 5 -->
-  <joint name="joint5" type="revolute">
-    <axis xyz="0 0 -1" rpy="0 0 0" />
-    <limit effort="1000.0" lower="${j5_lower_limit}" upper="${j5_upper_limit}" velocity="${j5_velocity_limit}"/>
-    <origin xyz="0 0 ${j4_length}" rpy="0 ${dh_j4_j5_roty} 0" />
-    <parent link="link4"/>
-    <child link="link5"/>
-    <dynamics damping="0.0" friction="0.0"/>
-  </joint>
-  <link name="link5">
-    <visual>
-      <geometry>
-        <mesh filename="package://rs_description/meshes/RS080N_J5.stl"/>
-      </geometry>
-      <material name="White"/>
-      <origin xyz="0 0 0" rpy="0 ${dh_j4_j5_roty*-1} 0"/>
-    </visual>
-    <collision>
-      <geometry>
-        <mesh filename="package://rs_description/meshes/RS080N_J5.stl"/>
-      </geometry>
-      <material name="White"/>
-      <origin xyz="0 0 0" rpy="0 ${dh_j4_j5_roty*-1} 0"/>
-    </collision>
-    <xacro:default_inertial mass="${j5_mass}"/>
-  </link>
-  <!-- Link 6 -->
-  <joint name="joint6" type="revolute">
-    <axis xyz="0 0 1" rpy="0 0 0" />
-    <limit effort="1000.0" lower="${j6_lower_limit}" upper="${j6_upper_limit}" velocity="${j6_velocity_limit}"/>
-    <origin xyz="${j5_length} 0 0" rpy="0 ${dh_j5_j6_roty} 0" />
-    <parent link="link5"/>
-    <child link="link6"/>
-    <dynamics damping="0.0" friction="0.0"/>
-  </joint>
-  <link name="link6">
-    <visual>
-      <geometry>
-        <mesh filename="package://rs_description/meshes/RS080N_J6.stl"/>
-      </geometry>
-      <material name="Black"/>
-      <origin xyz="0 0 0" rpy="0 0 0"/>
-    </visual>
-    <collision>
-      <geometry>
-        <mesh filename="package://rs_description/meshes/RS080N_J6.stl"/>
-      </geometry>
-      <material name="Black"/>
-      <origin xyz="0 0 0" rpy="0 0 0"/>
-    </collision>
-    <xacro:default_inertial mass="${j6_mass}"/>
-  </link>
 </robot>
